Commit message: Support for Gazebo Harmonic

File: robotnik_sensors/urdf/3d_lidar/robosense_helios_16p.urdf.xacro (robot description, xacro)
@@ -5,5 +5,5 @@
                        parent
                        *origin
-                       simulation:=false
+                       simulation:=true
                        node_name:=robosense_helios
                        node_namespace:=${None}
@@ -43,55 +43,34 @@
     </joint>
     <link name="${frame_prefix}link"/>
-    <xacro:if value="${simulation}">
-      <xacro:if value="${gpu}">
-        <xacro:property name="ray_type" value="gpu_ray" />
-      </xacro:if>
-      <xacro:unless value="${gpu}">
-        <xacro:property name="ray_type" value="ray" />
-      </xacro:unless>
       <gazebo reference="${frame_prefix}link">
-        <sensor type="${ray_type}" name="${frame_prefix}sensor">
-          <pose>0 0 0 0 0 0</pose>
-          <visualize>false</visualize>
-          <update_rate>10</update_rate>
-          <ray>
+        <sensor name='gpu_lidar' type='gpu_lidar'>
+          <pose relative_to='${frame_prefix}link'>0 0 0 0 0 0</pose>
+          <topic>${frame_prefix}sensor</topic>
+          <update_rate>20</update_rate>
+          <gz_frame_id>${frame_prefix}link</gz_frame_id>
+          <lidar>
             <scan>
               <horizontal>
-                <samples>1200</samples>
-                <resolution>1.0</resolution>
-                <min_angle>${-radians(180)}</min_angle>
-                <max_angle>${radians(180)}</max_angle>
+                <samples>450</samples> <!-- 900 -->
+                <resolution>1</resolution>
+                <min_angle>-3.141592</min_angle>
+                <max_angle>3.141592</max_angle>
               </horizontal>
               <vertical>
-                <samples>32</samples>
-                <resolution>1.0</resolution>
-                <min_angle>0.0</min_angle>
-                <max_angle>${radians(85)}</max_angle>
+                <samples>16</samples>
+                <resolution>1</resolution>
+                <min_angle>-0.261799</min_angle>
+                <max_angle>0.261799</max_angle>
               </vertical>
             </scan>
             <range>
-              <min>0.10</min>
-              <max>50</max>
-              <resolution>0.001</resolution>
+              <min>0.2</min>
+              <max>90.0</max>
+              <resolution>0.02</resolution>
             </range>
-            <noise>
-              <type>gaussian</type>
-              <mean>0.0</mean>
-              <stddev>0.00</stddev>
-            </noise>
-          </ray>
-          <plugin name="${node_name}" filename="libgazebo_ros_velodyne_laser.so">
-            <ros>
-              <namespace>${node_namespace}</namespace>
-            </ros>
-            <topicName>~/point_cloud</topicName>
-            <frameName>${node_namespace}/${frame_prefix}link</frameName>
-            <min_range>0.05</min_range>
-            <max_range>100.0</max_range>
-            <gaussianNoise>0.01</gaussianNoise>
-          </plugin>
+          </lidar>
+          <visualize>true</visualize>
         </sensor>
       </gazebo>
-    </xacro:if>
   </xacro:macro>
 </robot>

File: robotnik_sensors/urdf/3d_lidar/velodyne_vlp16.urdf.xacro (robot description, xacro)
@@ -42,13 +42,13 @@
     <xacro:if value="${simulation}">
       <xacro:if value="${gpu}">
-        <xacro:property name="ray_type" value="gpu_ray" />
+        <xacro:property name="ray_type" value="gpu_lidar" />
       </xacro:if>
       <xacro:unless value="${gpu}">
-        <xacro:property name="ray_type" value="ray" />
+        <xacro:property name="ray_type" value="lidar" />
       </xacro:unless>
       <gazebo reference="${frame_prefix}link">
         <sensor type="${ray_type}" name="${frame_prefix}sensor">
           <pose>0 0 0 0 0 0</pose>
-          <visualize>false</visualize>
+          <visualize>true</visualize>
           <update_rate>10</update_rate>
           <ray>
@@ -78,14 +78,4 @@
             </noise>
           </ray>
-          <plugin name="${node_name}" filename="libgazebo_ros_velodyne_laser.so">
-            <ros>
-              <namespace>${node_namespace}</namespace>
-            </ros>
-            <topicName>~/point_cloud</topicName>
-            <frameName>${node_namespace}/${frame_prefix}link</frameName>
-            <min_range>0.05</min_range>
-            <max_range>100.0</max_range>
-            <gaussianNoise>0.01</gaussianNoise>
-          </plugin>
         </sensor>
       </gazebo>

File: robotnik_sensors/urdf/all_sensors.urdf.xacro (robot description, xacro)
@@ -21,4 +21,5 @@
   <xacro:include filename="$(find robotnik_sensors)/urdf/3d_lidar/robosense_helios_16p.urdf.xacro" />
   <!-- IMUs -->
+  <xacro:include filename="$(find robotnik_sensors)/urdf/imu.urdf.xacro" />
   <xacro:include filename="$(find robotnik_sensors)/urdf/imu/vectornav.urdf.xacro" />
   <!-- GPS -->

File: robotnik_sensors/urdf/depth/stereolabs_generic.urdf.xacro (robot description, xacro)
@@ -6,5 +6,5 @@
                        *origin
                        model:=zed2
-                       simulation:=false
+                       simulation:=true
                        node_name:=stereolabs_generic
                        node_namespace:=${None}
@@ -57,5 +57,5 @@
       </inertial>
     </link>
-   <!-- Left camera -->
+    <!-- Left camera -->
     <joint name="${frame_prefix}color_left_joint" type="fixed">
       <origin xyz="0.0 0.06 0.0" rpy="0.0 0.0 0.0" />
@@ -83,5 +83,5 @@
     </joint>
     <link name="${frame_prefix}right_camera_optical_frame"/>
-    <!-- Depth image-->
+    <!-- Depth Camera-->
     <joint name="${frame_prefix}depth_joint" type="fixed">
       <origin xyz="0.0 0.0 0.0" rpy="0.0 0.0 0.0" />
@@ -96,113 +96,78 @@
     </joint>
     <link name="${frame_prefix}depth_optical_frame"/>
-    <xacro:if value="${simulation}">
-      <gazebo reference="${frame_prefix}right_camera_frame">
-        <sensor name="${frame_prefix}right_sensor" type="camera">
-          <pose>0.0 0.0 0.0 0.0 0.0 0.0</pose>
-          <visualize>false</visualize>
-          <update_rate>30</update_rate>
-          <camera>
-            <horizontal_fov>${radians(float(horizontal_fov))}</horizontal_fov>
-            <vertical_fov>${radians(float(vertical_fov))}</vertical_fov>
-            <image>
-              <width>${video_width}</width>
-              <height>${video_height}</height>
-              <format>R8G8B8</format>
-            </image>
-            <clip>
-              <near>0.10</near>
-              <far>100.0</far>
-            </clip>
-            <noise>
-              <type>gaussian</type>
-              <mean>0.0</mean>
-              <stddev>0.007</stddev>
-            </noise>
-          </camera>
-          <plugin name="${node_name}_right" filename="libgazebo_ros_camera.so">
-            <ros>
-              <namespace>${node_namespace}/${node_name}</namespace>
-              <remapping>right/image_raw:=right/image_raw_color</remapping>
-              <remapping>right/camera_info:=right/camera_info</remapping>
-            </ros>
-            <camera_name>right</camera_name>
-            <frame_name>${node_namespace}/${frame_prefix}right_camera_optical_frame</frame_name>
-          </plugin>
-        </sensor>
-      </gazebo>
-      <gazebo reference="${frame_prefix}left_camera_frame">
-        <sensor name="${frame_prefix}left_sensor" type="camera">
-          <pose>0.0 0.0 0.0 0.0 0.0 0.0</pose>
-          <visualize>false</visualize>
-          <update_rate>30</update_rate>
-          <camera>
-            <horizontal_fov>${radians(float(horizontal_fov))}</horizontal_fov>
-            <vertical_fov>${radians(float(vertical_fov))}</vertical_fov>
-            <image>
-              <width>${video_width}</width>
-              <height>${video_height}</height>
-              <format>R8G8B8</format>
-            </image>
-            <clip>
-              <near>0.10</near>
-              <far>100.0</far>
-            </clip>
-            <noise>
-              <type>gaussian</type>
-              <mean>0.0</mean>
-              <stddev>0.007</stddev>
-            </noise>
-          </camera>
-          <plugin name="${node_name}_left" filename="libgazebo_ros_camera.so">
-            <ros>
-              <namespace>${node_namespace}/${node_name}</namespace>
-              <remapping>left/image_raw:=left/image_raw_color</remapping>
-              <remapping>left/camera_info:=left/camera_info</remapping>
-            </ros>
-            <camera_name>left</camera_name>
-            <frame_name>${node_namespace}/${frame_prefix}left_camera_optical_frame</frame_name>
-          </plugin>
-        </sensor>
-      </gazebo>
-      <gazebo reference="${frame_prefix}depth_frame">
-        <sensor name="${frame_prefix}sensor" type="depth">
-          <pose>0.0 0.0 0.0 0.0 0.0 0.0</pose>
-          <visualize>false</visualize>
-          <update_rate>30</update_rate>
-          <camera>
-            <horizontal_fov>${radians(float(horizontal_fov))}</horizontal_fov>
-            <vertical_fov>${radians(float(vertical_fov))}</vertical_fov>
-            <image>
-              <width>${video_width}</width>
-              <height>${video_height}</height>
-              <format>B8G8R8</format>
-            </image>
-            <clip>
-              <near>0.05</near>
-              <far>100.0</far>
-            </clip>
-            <noise>
-              <type>gaussian</type>
-              <mean>0.0</mean>
-              <stddev>0.007</stddev>
-            </noise>
-          </camera>
-          <plugin name="${node_name}" filename="libgazebo_ros_camera.so">
-            <ros>
-              <namespace>${node_namespace}</namespace>
-              <remapping>~/image_raw:=${topic_prefix}rgb/image_raw_color</remapping>
-              <remapping>~/camera_info:=${topic_prefix}rgb/camera_info</remapping>
-              <remapping>~/points:=${topic_prefix}point_cloud/cloud_registered</remapping>
-              <remapping>~/depth/camera_info:=${topic_prefix}depth/camera_info</remapping>
-              <remapping>~/depth/image_raw:=${topic_prefix}depth/depth_registered</remapping>
-            </ros>
-            <camera_name>${node_name}</camera_name>
-            <frame_name>${node_namespace}/${frame_prefix}depth_optical_frame</frame_name>
-            <min_depth>${min_depth}</min_depth>
-            <max_depth>${max_depth}</max_depth>
-          </plugin>
-        </sensor>
-      </gazebo>
-    </xacro:if>
+    <!-- Right Camera Gazebo Definition -->
+    <gazebo reference="${frame_prefix}right_camera_frame">
+      <sensor name="${frame_prefix}right_sensor" type="camera">
+        <visualize>true</visualize>
+        <update_rate>30</update_rate>
+        <topic>/${frame_prefix}right/image</topic>
+        <camera>
+          <horizontal_fov>${radians(float(horizontal_fov))}</horizontal_fov>
+          <image>
+            <width>${video_width}</width>
+            <height>${video_height}</height>
+            <format>R8G8B8</format>
+          </image>
+          <clip>
+            <near>0.10</near>
+            <far>15.0</far>
+          </clip>
+          <noise>
+            <type>gaussian</type>
+            <mean>0.0</mean>
+            <stddev>0.007</stddev>
+          </noise>
+          <optical_frame_id>${frame_prefix}right_camera_frame</optical_frame_id>
+        </camera>
+      </sensor>
+    </gazebo>
+    <!-- Left Camera Gazebo Definition -->
+    <gazebo reference="${frame_prefix}left_camera_frame">
+      <sensor name="${frame_prefix}left_sensor" type="camera">
+        <visualize>false</visualize>
+        <update_rate>30</update_rate>
+        <topic>/${frame_prefix}left/image</topic>
+        <camera>
+          <horizontal_fov>${radians(float(horizontal_fov))}</horizontal_fov>
+          <image>
+            <width>${video_width}</width>
+            <height>${video_height}</height>
+            <format>R8G8B8</format>
+          </image>
+          <clip>
+            <near>0.10</near>
+            <far>15.0</far>
+          </clip>
+          <noise>
+            <type>gaussian</type>
+            <mean>0.0</mean>
+            <stddev>0.007</stddev>
+          </noise>
+          <optical_frame_id>${frame_prefix}left_camera_frame</optical_frame_id>
+        </camera>
+      </sensor>
+    </gazebo>
+    <!-- Depth Camera Gazebo Definition -->
+    <gazebo reference="${frame_prefix}depth_frame">
+      <sensor name="rgbd_camera" type="rgbd_camera">
+        <camera>
+          <horizontal_fov>${radians(float(horizontal_fov))}</horizontal_fov>
+          <image>
+            <width>${video_width}</width>
+            <height>${video_height}</height>
+          </image>
+          <clip>
+            <near>${min_depth}</near>
+            <far>${max_depth}</far>
+          </clip>
+          <optical_frame_id>${frame_prefix}depth_frame</optical_frame_id>
+        </camera>
+        <always_on>1</always_on>
+        <update_rate>20</update_rate>
+        <visualize>true</visualize>
+        <topic>/${frame_prefix}depth_camera</topic>
+        <gz_frame_id>${frame_prefix}depth_frame</gz_frame_id>
+      </sensor>
+    </gazebo>
   </xacro:macro>
 </robot>

File: robotnik_sensors/urdf/depth/stereolabs_zed2.urdf.xacro (robot description, xacro)
@@ -5,5 +5,5 @@
                        parent
                        *origin
-                       simulation:=false
+                       simulation:=true
                        node_namespace:=stereolabs_zed2
                        node_name:=stereolabs_zed2
@@ -18,6 +18,6 @@
                                      horizontal_fov="110"
                                      vertical_fov="70"
-                                     video_width="1920"
-                                     video_height="1080"
+                                     video_width="960"
+                                     video_height="540"
                                      video_fps="30"
                                      min_depth="0.2"

File: robotnik_sensors/urdf/gps/gps.urdf.xacro (robot description, xacro)
@@ -42,46 +42,11 @@
 	  </gazebo>
     <gazebo reference="${frame_prefix}base_link">
-      <sensor type="gps" name="${frame_prefix}sensor">
-        <always_on>true</always_on>
+      <sensor name="${frame_prefix}sensor" type="navsat">
+        <always_on>1</always_on>
         <update_rate>${update_rate}</update_rate>
-        <gps>
-          <position_sensing>
-            <horizontal>
-              <noise type="gaussian">
-                <mean>0.0</mean>
-                <stddev>0.1</stddev>
-              </noise>
-            </horizontal>
-            <vertical>
-              <noise type="gaussian">
-                <mean>0.0</mean>
-                <stddev>0.1</stddev>
-              </noise>
-            </vertical>
-          </position_sensing>
-          <vertical_sensing>
-            <horizontal>
-              <noise type="gaussian">
-                <mean>0.0</mean>
-                <stddev>0.1</stddev>
-              </noise>
-            </horizontal>
-            <vertical>
-              <noise type="gaussian">
-                <mean>0.0</mean>
-                <stddev>0.1</stddev>
-              </noise>
-            </vertical>
-          </vertical_sensing>
-        </gps>
-        <plugin name="${node_name}" filename="libgazebo_ros_gps_sensor.so">
-          <ros>
-            <namespace>${node_namespace}</namespace>
-            <remapping>~/out:=${topic_prefix}fix</remapping>
-            <remapping>~/vel:=${topic_prefix}vel</remapping>
-          </ros>
-        </plugin>
+        <topic>/robot/gps/fix</topic>
+        <gz_frame_id>${frame_prefix}base_link</gz_frame_id>
       </sensor>
-	  </gazebo>
+    </gazebo>
   </xacro:macro>
 </robot>

File: robotnik_sensors/urdf/imu.urdf.xacro (robot description, xacro)
@@ -4,5 +4,4 @@
 	  <joint name="${prefix}_joint" type="fixed">
 	      <axis xyz="1 0 0"/>
-	      <!--origin xyz="0 0 0.2825"/-->
 	      <xacro:insert_block name="origin"/>
 	      <parent link="${parent}"/>
@@ -21,39 +20,12 @@
 	        </geometry>
 	      </visual>
-	      <!--collision>
-	        <origin rpy="0 0 0" xyz="0 0 0"/>
-	        <geometry>
-	          <box size="0.001 0.001 0.001"/>
-	        </geometry>
-	      </collision-->
 	  </link>
-	  <!--<gazebo>-->
-		<!--<plugin name="${prefix}_controller" filename="libgazebo_ros_imu.so">-->
-		   <!--<topicName>${ns}imu/data</topicName>-->
-		   <!--<serviceName>imu/service</serviceName>-->
-		   <!--<bodyName>${prefix}_link</bodyName>-->
-		   <!--<updateRateHZ>50.0</updateRateHZ>-->
-		   <!--<gaussianNoise>0.0</gaussianNoise>-->
-		<!--</plugin>-->
-	  <!--</gazebo>-->
- <gazebo reference="${prefix}_link">
-    <gravity>true</gravity>
-    <sensor name="${prefix}_imu_sensor" type="imu">
-      <always_on>true</always_on>
-      <update_rate>100</update_rate>
-      <visualize>true</visualize>
-      <topic>__default_topic__</topic>
-      <plugin filename="libgazebo_ros_imu_sensor.so" name="${prefix}_imu_plugin">
-        <topicName>${topic}</topicName>
-		<bodyName>${prefix}_link</bodyName>
-        <updateRateHZ>100.0</updateRateHZ>
-        <gaussianNoise>0.0</gaussianNoise>
-        <xyzOffset>0 0 0</xyzOffset>
-        <rpyOffset>0 0 0</rpyOffset>
-		<frameName>${prefix}_link</frameName>
-      </plugin>
-      <pose>0 0 0 0 0 0</pose>
-    </sensor>
-  </gazebo>
+    <gazebo reference="${prefix}_link">
+      <sensor name="${prefix}_sensor" type="imu">
+        <always_on>1</always_on>
+        <update_rate>30</update_rate>
+        <topic>${topic}</topic>
+      </sensor>
+    </gazebo>
   </xacro:macro>
 </robot>

File: robotnik_sensors/urdf/imu/vectornav.urdf.xacro (robot description, xacro)
@@ -114,12 +114,4 @@
           </linear_acceleration>
         </imu>
-        <plugin name="${node_name}" filename="libgazebo_ros_imu_sensor.so">
-          <ros>
-            <namespace>${node_namespace}</namespace>
-            <remapping>~/out:=${topic_prefix}data</remapping>
-          </ros>
-          <initial_orientation_as_reference>false</initial_orientation_as_reference>
-          <frame_name>${node_namespace}/${frame_prefix}link</frame_name>
-        </plugin>
       </sensor>
     </gazebo>

Commit message: Lidar, GPS and cameras were modified

File: robotnik_sensors/urdf/3d_lidar/robosense_helios_16p.urdf.xacro (robot description, xacro)
@@ -10,10 +10,10 @@
                        topic_prefix:=~/
                        gpu:=true">
-    <joint name="${frame_prefix}base_joint" type="fixed">
+    <joint name="${frame_prefix}_base_joint" type="fixed">
       <xacro:insert_block name="origin" />
       <parent link="${parent}"/>
-      <child link="${frame_prefix}base_link"/>
+      <child link="${frame_prefix}_base_link"/>
     </joint>
-    <link name="${frame_prefix}base_link">
+    <link name="${frame_prefix}_base_link">
       <collision>
         <origin xyz="0 0 0" rpy="0 0 0"/>
@@ -37,16 +37,16 @@
       </inertial>
     </link>
-    <joint name="${frame_prefix}joint" type="fixed">
-      <parent link="${frame_prefix}base_link"/>
-      <child link="${frame_prefix}link"/>
+    <joint name="${frame_prefix}_joint" type="fixed">
+      <parent link="${frame_prefix}_base_link"/>
+      <child link="${frame_prefix}_link"/>
       <origin xyz="0.0 0 0.0635" rpy="0 0 0"/>
     </joint>
-    <link name="${frame_prefix}link"/>
-      <gazebo reference="${frame_prefix}link">
+    <link name="${frame_prefix}_link"/>
+      <gazebo reference="${frame_prefix}_link">
         <sensor name='gpu_lidar' type='gpu_lidar'>
-          <pose relative_to='${frame_prefix}link'>0 0 0 0 0 0</pose>
-          <topic>${frame_prefix}sensor</topic>
+          <pose relative_to='${frame_prefix}_link'>0 0 0 0 0 0</pose>
+          <topic>${frame_prefix}</topic>
           <update_rate>20</update_rate>
-          <gz_frame_id>${frame_prefix}link</gz_frame_id>
+          <gz_frame_id>${frame_prefix}_link</gz_frame_id>
           <ray>
             <scan>

File: robotnik_sensors/urdf/depth/stereolabs_zed2.urdf.xacro (robot description, xacro)
@@ -18,10 +18,11 @@
                                      horizontal_fov="110"
                                      vertical_fov="70"
-                                     video_width="960"
-                                     video_height="540"
+                                     video_width="640"
+                                     video_height="360"
                                      video_fps="30"
                                      min_depth="0.2"
                                      max_depth="20.0">
       <xacro:insert_block name="origin" />
+      <!-- 960 x 540 -->
     </xacro:sensor_stereolabs_generic>
   </xacro:macro>

File: robotnik_sensors/urdf/gps/gps.urdf.xacro (robot description, xacro)
@@ -9,5 +9,5 @@
                        node_namespace:=${None}
                        topic_prefix:=~/
-                       update_rate:=5.0">
+                       update_rate:=1.0">
 	  <joint name="${frame_prefix}joint" type="fixed">
 	    <xacro:insert_block name="origin"/>
@@ -45,5 +45,5 @@
         <always_on>1</always_on>
         <update_rate>${update_rate}</update_rate>
-        <topic>/robot/gps/fix</topic>
+        <topic>gps/fix</topic>
         <gz_frame_id>${frame_prefix}base_link</gz_frame_id>
       </sensor>
