Commit message: fix: removed double underscore for gps__link, and added imu_link frame name tf to sim frame

File: robotnik_sensors/urdf/gps/gps.urdf.xacro (robot description, xacro)
@@ -13,7 +13,7 @@
 	    <xacro:insert_block name="origin"/>
 	    <parent link="${parent}"/>
-	    <child link="${frame_prefix}base_link"/>
+	    <child link="${frame_prefix}link"/>
 	  </joint>
-	  <link name="${frame_prefix}base_link">
+	  <link name="${frame_prefix}link">
       <inertial>
         <origin xyz="0.0 0 0.015" rpy="0 0 0" />
@@ -37,14 +37,14 @@
 	    </collision>
 	  </link>
-	  <gazebo reference="${frame_prefix}base_link">
+	  <gazebo reference="${frame_prefix}link">
 	    <material>Gazebo/White</material>
 	    <gravity>true</gravity>
 	  </gazebo>
-    <gazebo reference="${frame_prefix}base_link">
+    <gazebo reference="${frame_prefix}link">
       <sensor name="${frame_prefix}sensor" type="navsat">
         <always_on>1</always_on>
         <update_rate>${update_rate}</update_rate>
         <topic>gps/fix</topic>
-        <gz_frame_id>${frame_prefix}base_link</gz_frame_id>
+        <gz_frame_id>${frame_prefix}link</gz_frame_id>
       </sensor>
     </gazebo>

File: robotnik_sensors/urdf/gps_with_mast.urdf.xacro (robot description, xacro)
@@ -6,5 +6,5 @@
   <xacro:macro name="sensor_gps_with_mast" params="prefix parent *origin gps_latitude:=^|39.5080331 gps_longitude:=^|-0.4619816 update_rate:=^|5">
 	  <!-- MAST OF THE ANTENNA GPS -->
-	  <joint name="${prefix}_joint" type="fixed">
+	  <joint name="${prefix}_base_joint" type="fixed">
 	    <axis xyz="0 1 0"/>
 	    <xacro:insert_block name="origin"/>
@@ -37,5 +37,5 @@
 	    <axis xyz="0 1 0"/>
 	    <parent link="${prefix}_mast_base_link"/>
-	    <child link="${prefix}_base_link"/>
+	    <child link="${prefix}_link"/>
 	    <origin xyz="0 0 ${mast_height/2.0}" rpy="0 0 0" />
 	  </joint>
@@ -45,5 +45,5 @@
 	  </gazebo>
       <!-- ANTENNA GPS -->
-	  <link name="${prefix}_base_link">
+	  <link name="${prefix}_link">
 	    <inertial>
 			<origin xyz="0.0 0 0.015" rpy="0 0 0" />
@@ -67,5 +67,5 @@
 	    </collision>
 	  </link>
-	  <gazebo reference="${prefix}_base_link">
+	  <gazebo reference="${prefix}_link">
 	    <material>Gazebo/White</material>
 	    <gravity>true</gravity>
@@ -75,6 +75,6 @@
         <alwaysOn>1</alwaysOn>
         <updateRate>${update_rate}</updateRate>
-        <bodyName>${prefix}_base_link</bodyName> <!-- must be the link of the gps device, not the base_link or base_footprint -->
-        <frameId>${prefix}_base_link</frameId>   <!-- which frame_id would be on the published message -->
+        <bodyName>${prefix}_link</bodyName> <!-- must be the link of the gps device, not the base_link or base_footprint -->
+        <frameId>${prefix}_link</frameId>   <!-- which frame_id would be on the published message -->
         <topicName>gps/fix</topicName>
         <!-- GPS coordinates -->

File: robotnik_sensors/urdf/imu.urdf.xacro (robot description, xacro)
@@ -21,4 +21,10 @@
 	      </visual>
 	  </link>
+    <joint name="${prefix}_gazebo_frame_joint" type="fixed">
+      <origin xyz="0 0 0" rpy="0 0 0"/>
+      <parent link="${prefix}_link"/>
+      <child link="summit_xl/base_footprint/imu_sensor"/>
+    </joint>
+    <link name="summit_xl/base_footprint/imu_sensor"/>
     <gazebo reference="${prefix}_link">
       <sensor name="${prefix}_sensor" type="imu">
